File: dsn/main/Luxeon Rebel Controller Board.brd (EAGLE design)
At the start: 63.5 x 63.5 mm, 37 parts, among them IC1 LM7805, IC2 ATMEGA328P-PU, IC3 SN74AHC1G125DCKR, IC4 SN74AHC1G125DCKR, Q1 2N2222, Q2 2N2222, Q3 2N2222

Commit message: fixed names
Parts:
- R7: value 5K -> 4.7K
Connections:
- net N$4 renamed VIN
Changed lines of the file:
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@@
 <attribute name="NAME" x="44.461321875" y="15.65341875" size="0.8128" layer="25" ratio="10" rot="SR45"/>
 </element>
-<element name="R7" library="SparkFun-Passives" package="0603-RES" value="5K" x="47.6" y="21.7" smashed="yes" rot="R90">
+<element name="R7" library="SparkFun-Passives" package="0603-RES" value="4.7K" x="47.6" y="21.7" smashed="yes" rot="R90">
 <attribute name="NAME" x="49.038" y="20.311" size="0.4064" layer="25" font="vector" rot="R90"/>
 </element>
@@
 <wire x1="34.29" y1="49.79" x2="34.29" y2="53.34" width="0.6096" layer="1"/>
 </signal>
-<signal name="N$4">
+<signal name="VIN">
 <contactref element="IC1" pad="IN"/>
 <contactref element="JP4" pad="5"/>
