File: dsn/main/Luxeon Rebel Controller Board.sch (EAGLE design)
At the start: 35 parts, among them IC1 LM7805, IC2 ATMEGA328P-PU, IC3 SN74AHC1G125DCKR, IC4 SN74AHC1G125DCKR, Q1 2N2222, Q2 2N2222, Q3 2N2222

Commit message: fixed names
Parts:
- R7: value 5K -> 4.7K
Connections:
- net N$4 renamed VIN
Other:
- moved on the sheet: ADC, GPIO, GPIOB, IC3, IC4, R7, SJ2, SPP-BT, XTAL
